File: DataloggerSMNViento/_autosave-DataloggerSMNViento.kicad_sch (KiCad schematic)
At the start: 0 parts

Commit message: Agrego el esquemático del poncho Datalogger para SCTV
Other:
- company: Proyecto CIAA - COMPUTADORA INDUSTRIAL ABIERTA ARGENTINA -> Servicio Meteorológico Nacional - FIUBA - UBA
- title: Poncho Grande - Modelo - Ejemplo - Template -> Datalogger para SCTV
