File: DataloggerSMNViento/_autosave-conector_poncho.kicad_sch (KiCad schematic)
At the start: 1 part

Commit message: Agrego el esquemático del poncho Datalogger para SCTV
Other:
- company: Compañia: Servicio Meteorologico Nacional - Universidad de Buenos Aires -> Servicio Meteorológico Nacional - FIUBA - UBA
- title: Poncho Grande - Datalogger SMN Viento -> Datalogger para SCTV
Changed lines of the file:
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@@
   (paper "A4")
   (title_block
-    (title "Poncho Grande - Datalogger SMN Viento")
-    (date "2015-10-06")
+    (title "Datalogger para SCTV")
+    (date "2023-10-20")
     (rev "1.0")
-    (company "Compañia: Servicio Meteorologico Nacional - Universidad de Buenos Aires")
-    (comment 1 "https://github.com/ciaa/Ponchos/tree/master/modelos/doc")
-    (comment 2 "Licencia: Ver Licencia.txt UBA")
-    (comment 3 "Autor del poncho: Cristian Zozimo Aranda Cordero. Ver directorio \"doc\"")
-    (comment 4 "CÓDIGO PONCHO:")
+    (company "Servicio Meteorológico Nacional - FIUBA - UBA")
+    (comment 1 "poner repo")
+    (comment 2 "Autores y Licencia del poncho: Cristian Aranda (FIUBA), ver archivo licence.txt")
+    (comment 3 "Autor del poncho: Cristian Zozimo Aranda Cordero.  Ver directorio \"doc\"")
+    (comment 4 "CÓDIGO PONCHO: DT1")
   )
   (junction (at 171.45 66.04) (diameter 0) (color 0 0 0 0)
