File: DataloggerSMNViento/principal.kicad_sch (KiCad schematic)
At the start: 21 parts, among them P1 CONN_01X06, P10 CONN_01X12, P11 CONN_02X20, P12 CONN_02X20, P13 CONN_01X20, P14 CONN_02X20, P15 CONN_01X20, P16 CONN_01X19, P17 CONN_01X20, P18 CONN_02X20, P19 CONN_01X20, P2 CONN_01X06, P20 CONN_02X20, P21 CONN_02X20, P3 CONN_02X12, P4 CONN_02X12, P5 CONN_02X12, P6 CONN_02X12, P7 CONN_01X12, P8 CONN_01X12, P9 CONN_01X12

Commit message: Agrego modificaciones al poncho de la EDU CIAA, también agrego una simulacion del circuito para tomar la tensión del ADC del tunnel
Parts:
- removed P1, P2: CONN_01X06, mod:bornier6, symbol Misc_Poncho_Grande:CONN_01X06
- removed P10, P7, P8, P9: CONN_01X12, Pin_Headers:Pin_Header_Straight_1x12, symbol Misc_Poncho_Grande:CONN_01X12
- removed P11, P12, P14, P18, P20, P21: CONN_02X20, Pin_Headers:Pin_Header_Straight_2x20, symbol Misc_Poncho_Grande:CONN_02X20
- removed P13, P19: CONN_01X20, Pin_Headers:Pin_Header_Straight_2x12, symbol Misc_Poncho_Grande:CONN_02X12
- removed P15, P17: CONN_01X20, Pin_Headers:Pin_Header_Straight_1x20, symbol Misc_Poncho_Grande:CONN_01X20
- removed P16: CONN_01X19, Pin_Headers:Pin_Header_Straight_1x19, symbol Misc_Poncho_Grande:CONN_01X19
- removed P3, P4, P5, P6: CONN_02X12, Pin_Headers:Pin_Header_Straight_2x12, symbol Misc_Poncho_Grande:CONN_02X12
Connections:
- no-connect marks 43 -> 0
