File: Osciloscopio/Display.sch (KiCad schematic (older format))
At the start: 8 parts

Commit message: Agrego modificaciones al poncho de la EDU CIAA, también agrego una simulacion del circuito para tomar la tensión del ADC del tunnel
Parts:
- removed D5: Display, osc:Display, symbol Display
- removed R20, R21, R22, R23, R24, R25, R26: 33, osc:R_0805_HandSoldering, symbol R
Connections:
- net labels removed: +5VP, GND
