File: Osciloscopio/conector_poncho.sch (KiCad schematic (older format))
At the start: 1 part

Commit message: Agrego modificaciones al poncho de la EDU CIAA, también agrego una simulacion del circuito para tomar la tensión del ADC del tunnel
Parts:
- removed XA1: Conn_Poncho2P_2x_20x2, osc:poncho_grande, symbol Conn_Poncho2P_2x_20x2
