File: Osciloscopio/osciloscopio.sch (KiCad schematic (older format))
At the start: 35 parts, among them P1 BNC, Q1 BC557, Q2 BC557, Q3 BC557, Q4 BC557, U4 TL082, U5 CD4066

Commit message: Agrego modificaciones al poncho de la EDU CIAA, también agrego una simulacion del circuito para tomar la tensión del ADC del tunnel
Parts:
- removed C10, C11, C12, C14: 100nF, osc:C_0805_HandSoldering, symbol C
- removed D1, D2, D3, D4: BAT54, osc:SOT-323, symbol D_Schottky_Small
- removed P1: BNC, osc:BNC_Socket_TYCO-AMP_LargePads, symbol BNC
- removed Q1, Q2, Q3, Q4: BC557, osc:TO-92_Inline_Wide, symbol Q_PNP_CBE
- removed R1: 10k, osc:R_0805_HandSoldering, symbol R
- removed R10, R11, R8, R9: 47k, osc:R_0805_HandSoldering, symbol R
- removed R12, R17, R19: 56k, osc:R_0805_HandSoldering, symbol R
- removed R13: 18k, osc:R_0805_HandSoldering, symbol R
- removed R14: 5k6, osc:R_0805_HandSoldering, symbol R
- removed R15: 1k8, osc:R_0805_HandSoldering, symbol R
- removed R16: 150k, osc:R_0805_HandSoldering, symbol R
- removed R2, R3, R4, R5, R7: 100k, osc:R_0805_HandSoldering, symbol R
- removed R6: 910k, osc:R_0805_HandSoldering, symbol R
- removed RV1: 10k, osc:Potentiometer_Alps-RK16-single, symbol POT
- removed RV2: 150k, osc:Potentiometer_Bourns_3296W_3-8Zoll_Inline_ScrewUp, symbol POT
- removed U4: TL082, osc:DIP-8_W7.62mm_LongPads, symbol TL082
- removed U5: CD4066, osc:DIP-14_W7.62mm_LongPads, symbol CD4066
Connections:
- net labels removed: +3.3VADC, +3.3VP, +5VA, -5VA, GNDA
- wire segments 106 -> 137
