File: Osciloscopio/power.sch (KiCad schematic (older format))
At the start: 14 parts, among them U1 MAX232, U2 78L05, U3 79L05

Commit message: Agrego modificaciones al poncho de la EDU CIAA, también agrego una simulacion del circuito para tomar la tensión del ADC del tunnel
Parts:
- removed C1, C2, C3, C4, C5: 1uF, osc:C_Radial_D5_L11_P2, symbol CP
- removed C6, C7, C8, C9: 100nF, osc:C_0805_HandSoldering, symbol C
- removed FB1, FB2: HZ0805E601R-10, osc:R_0805_HandSoldering, symbol FILTER
- removed U1: MAX232, osc:DIP-16_W7.62mm_LongPads, symbol MAX232
- removed U2: 78L05, osc:TO-92_Inline_Wide, symbol 78L05
- removed U3: 79L05, osc:TO-92_Inline_Wide, symbol 79L05
Connections:
- net labels removed: +5VA, +5VP, -5VA, GND
- wire segments 49 -> 67
